File: hardware/openscex-bare.kicad_pcb (KiCad board)
At the start: 2 copper layers, 35.6 x 21.6 mm, 8 parts, among them U1 ATtiny85-20PU

Commit message: feat(hardware): add a RESET pull-up to every board
The mini and bare boards now hold pin 1 high with a 10 kOhm pull-up,
as the carrier already did. The chip's own pull-up is 30 to 60 kOhm,
weak against noise coupled in from the console, and a spurious reset
costs the region check of the disc being read. Any ISP programmer
still overrides it.
Parts:
- added R1: 10k, Resistor_THT:R_Axial_DIN0204_L3.6mm_D1.6mm_P5.08mm_Horizontal, F.Cu at (124.5, 105.0)
Connections:
- U1 pad 1: unconnected-(U1-~{RESET}/PB5-Pad1) -> /RST
Routing:
- net /RST: track 0.00 -> 5.41 mm
- net /VCC: track 13.9 -> 18.3 mm
- net /GND: vias 35 -> 31

Commit message: feat(hardware): name datasheet-checked parts
Every BOM line now names an exact manufacturer part, each checked
against its own datasheet: Microchip ATTINY85-20PU in a TE
1-2199298-2 socket, KEMET C315C104K5R5TA, Panasonic EEU-FC1A101S,
Vishay MBA0204 resistors, onsemi 2N3904RLRAG and 1N4148TR,
Kingbright WP710A10ID, CTS 206-2ST, Same Sky CMI-1295IC-0385T and
Wurth 61200621621.

C1 moves to a 4.0 x 2.5 mm footprint that fits the KEMET body. A
project footprint library, hardware/openscex.pretty, carries the hole
sizes the Wurth header and the buzzer datasheets recommend, 1.1 mm and
0.8 mm in 2 mm pads.
Parts:
- C1: footprint Capacitor_THT:C_Disc_D3.0mm_W1.6mm_P2.50mm -> Capacitor_THT:C_Rect_L4.0mm_W2.5mm_P2.50mm
- moved C1 0.38 mm to (122.6, 114.0)
Routing:
- net /VCC: track 18.3 -> 19.0 mm
