File: hardware/openscex.kicad_sch (KiCad schematic)
At the start: 12 parts, among them J1 ISP, U1 ATtiny85-20PU

Commit message: feat: one symmetric board with optional headers
The carrier, mini and bare boards become one board. The socket, a
100 nF ceramic, a 220 uF bulk capacitor and the 10 kOhm RESET pull-up
are always fitted; a keyed ISP header, a keyed JST XH 3-pin indicator
header and a 6-pin serial header for the trace image are optional and
marked on the silkscreen and in the BOM's Fit column.

The indicator header carries GND, VCC and PB3 in servo order, so a
reversed plug never reverses power, and takes a cable to whatever
indicator the builder chooses: an LED with its resistor, an active
buzzer or a board of their own. The bulk capacitor holds the supply
through such a load's pulses. The board carries no LED, buzzer or
switch of its own.

The layout is symmetric about the vertical centre line, every track
is routed at the widest width that fits, 1.0 mm here, and every bend
is a tangent arc. AGENTS rules 7 and 16 state both, and the board
test checks the symmetry.
Parts:
- removed D1: LED red 3 mm, LED_THT:LED_D3.0mm, symbol Device:LED
- removed R2: 10k, Resistor_THT:R_Axial_DIN0204_L3.6mm_D1.6mm_P5.08mm_Horizontal, symbol Device:R
- added C2: 220uF, Capacitor_THT:CP_Radial_D6.3mm_P2.50mm, symbol Device:C_Polarized
- added J2: IND, Connector_JST:JST_XH_B3B-XH-A_1x03_P2.50mm_Vertical, symbol Connector_Generic:Conn_01x03
- added J3: SERIAL, Connector_PinHeader_2.54mm:PinHeader_1x06_P2.54mm_Vertical, symbol Connector_Generic:Conn_01x06
- C1, TP1, TP2, TP3, TP4, TP5, TP6, U1: Fit (none) -> always
- J1: Fit (none) -> optional
- R1: value 1k -> 10k; Fit (none) -> always; Part Vishay MBA02040C1001FC100, 1 kOhm 1 % 0.4 W, 0204 -> Vishay MBA02040C1002FC100, 10 kOhm 1 % 0.4 W, 0204
Connections:
- net LED_A is gone; now on net VCC: R1.2
- net GND: now also C2.2, J2.1 (Pin_1), J3.1 (Pin_1)
- net PB3: now also J2.3 (Pin_3), J3.5 (Pin_5); no longer R1.1
- net RST: now also R1.1
- net VCC: now also C2.1, J2.2 (Pin_2)
- no-connect marks 0 -> 4
Other:
- title: openscex mini -> openscex
- moved on the sheet: R1
